File: YAsixtyfive02.kicad_sch (KiCad schematic)
At the start: 59 parts, among them J1 ~{NMI}, J2 Aux 5VDC, J3 Power 5V, J4 Expansion Bus, J7 GND, J8 FTDI Serial2USB, SW1 RESET, SW2 SW_Push_DPDT, U1 WD65C02, U10 74LS138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

Commit message: rev. 1.6.1 minor pcb routing tweaks all IO in the connector
Parts:
- C8: footprint Capacitor_THT:CP_Radial_D8.0mm_P3.80mm -> Capacitor_THT:CP_Radial_D6.3mm_P2.50mm
- TP1, TP2, TP7: footprint TestPoint:TestPoint_THTPad_2.0x2.0mm_Drill1.0mm -> TestPoint:TestPoint_THTPad_1.5x1.5mm_Drill0.7mm
Changed lines of the file:
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@@
     (title "YAsixfive02 SBC")
     (date "2022-10-11")
-    (rev "1.6.0")
+    (rev "1.6.1")
     (company "(c) Mariano Luna")
   )
@@
       (effects (font (size 1.27 1.27)) (justify left))
     )
-    (property "Footprint" "Capacitor_THT:CP_Radial_D8.0mm_P3.80mm" (id 2) (at 269.24 142.5448 0)
+    (property "Footprint" "Capacitor_THT:CP_Radial_D6.3mm_P2.50mm" (id 2) (at 269.24 142.5448 0)
       (effects (font (size 1.27 1.27)) hide)
     )
@@
       (effects (font (size 1.27 1.27)) (justify left))
     )
-    (property "Footprint" "TestPoint:TestPoint_THTPad_2.0x2.0mm_Drill1.0mm" (id 2) (at 87.63 35.56 0)
+    (property "Footprint" "TestPoint:TestPoint_THTPad_1.5x1.5mm_Drill0.7mm" (id 2) (at 87.63 35.56 0)
       (effects (font (size 1.27 1.27)) hide)
     )
@@
     (property "Reference" "TP2" (id 0) (at 226.06 85.09 90))
     (property "Value" "~{RESET}" (id 1) (at 226.06 87.63 90))
-    (property "Footprint" "TestPoint:TestPoint_THTPad_2.0x2.0mm_Drill1.0mm" (id 2) (at 231.14 81.28 0)
+    (property "Footprint" "TestPoint:TestPoint_THTPad_1.5x1.5mm_Drill0.7mm" (id 2) (at 231.14 81.28 0)
       (effects (font (size 1.27 1.27)) hide)
     )
@@
       (effects (font (size 1.27 1.27)) (justify left))
     )
-    (property "Footprint" "TestPoint:TestPoint_THTPad_2.0x2.0mm_Drill1.0mm" (id 2) (at 87.63 101.6 0)
+    (property "Footprint" "TestPoint:TestPoint_THTPad_1.5x1.5mm_Drill0.7mm" (id 2) (at 87.63 101.6 0)
       (effects (font (size 1.27 1.27)) hide)
     )
@@
     )
     (path "/00000000-0000-0000-0000-00006163f681"
-      (reference "C8") (unit 1) (value "100uF") (footprint "Capacitor_THT:CP_Radial_D8.0mm_P3.80mm")
+      (reference "C8") (unit 1) (value "100uF") (footprint "Capacitor_THT:CP_Radial_D6.3mm_P2.50mm")
     )
     (path "/103b9359-a2d1-4e8c-9f92-4774d1636b0a"
@@
     )
     (path "/00000000-0000-0000-0000-00006349f52f"
-      (reference "TP1") (unit 1) (value "CLK") (footprint "TestPoint:TestPoint_THTPad_2.0x2.0mm_Drill1.0mm")
+      (reference "TP1") (unit 1) (value "CLK") (footprint "TestPoint:TestPoint_THTPad_1.5x1.5mm_Drill0.7mm")
     )
     (path "/00000000-0000-0000-0000-000063d64eab"
-      (reference "TP2") (unit 1) (value "~{RESET}") (footprint "TestPoint:TestPoint_THTPad_2.0x2.0mm_Drill1.0mm")
+      (reference "TP2") (unit 1) (value "~{RESET}") (footprint "TestPoint:TestPoint_THTPad_1.5x1.5mm_Drill0.7mm")
     )
     (path "/75f85b84-9777-4d8b-a0f4-27c0e653b059"
@@
     )
     (path "/3f7b3ccb-d9de-421f-9547-3f5e141f058b"
-      (reference "TP7") (unit 1) (value "ACIA_CLK") (footprint "TestPoint:TestPoint_THTPad_2.0x2.0mm_Drill1.0mm")
+      (reference "TP7") (unit 1) (value "ACIA_CLK") (footprint "TestPoint:TestPoint_THTPad_1.5x1.5mm_Drill0.7mm")
     )
     (path "/00000000-0000-0000-0000-0000612219a0"
